Commit message: lbr_ prefix

File: urdf/lbr_med7_r800.urdf.xacro (robot description, xacro)
@@ -3,10 +3,10 @@
 <robot name="med7" xmlns:xacro="http://www.ros.org/wiki/xacro">
     <!-- include the Med 7 R800 macro -->
-    <xacro:include filename="$(find med7_r800_description)/urdf/med7_r800_macro.xacro" />
+    <xacro:include filename="$(find lbr_med7_r800_description)/urdf/lbr_med7_r800_macro.xacro" />
     <!-- arguments -->
     <xacro:arg name="robot_name" default="lbr" />
     <xacro:arg
         name="joint_limits_path"
-        default="$(find med7_r800_description)/config/joint_limits.yaml" />
+        default="$(find lbr_med7_r800_description)/config/joint_limits.yaml" />
     <!-- Med 7 R800 description -->
     <xacro:med7_r800

File: urdf/lbr_med7_r800_macro.xacro (robot description, xacro)
@@ -3,5 +3,5 @@
     <!-- robot as extracted via https://github.com/syuntoku14/fusion2urdf -->
     <xacro:macro name="med7_r800"
-        params="robot_name:=^|lbr joint_limits_path:=^|'$(find med7_r800_description)/config/joint_limits.yaml'">
+        params="robot_name:=^|lbr joint_limits_path:=^|'$(find lbr_med7_r800_description)/config/joint_limits.yaml'">
         <!-- load joint limits via yaml -->
         <xacro:property name="joint_limits" value="${xacro.load_yaml(joint_limits_path)}" />
@@ -21,5 +21,5 @@
                 <origin rpy="0 0 0" xyz="0 0 0" />
                 <geometry>
-                    <mesh filename="package://med7_r800_description/meshes/visual/link_0.dae" />
+                    <mesh filename="package://lbr_med7_r800_description/meshes/visual/link_0.dae" />
                 </geometry>
             </visual>
@@ -27,5 +27,5 @@
                 <origin rpy="0 0 0" xyz="0 0 0" />
                 <geometry>
-                    <mesh filename="package://med7_r800_description/meshes/collision/link_0.stl" />
+                    <mesh filename="package://lbr_med7_r800_description/meshes/collision/link_0.stl" />
                 </geometry>
             </collision>
@@ -58,5 +58,5 @@
                 <origin rpy="0 0 0" xyz="0.0 0.0 -0.1475" />
                 <geometry>
-                    <mesh filename="package://med7_r800_description/meshes/visual/link_1.dae" />
+                    <mesh filename="package://lbr_med7_r800_description/meshes/visual/link_1.dae" />
                 </geometry>
             </visual>
@@ -64,5 +64,5 @@
                 <origin rpy="0 0 0" xyz="0.0 0.0 -0.1475" />
                 <geometry>
-                    <mesh filename="package://med7_r800_description/meshes/collision/link_1.stl" />
+                    <mesh filename="package://lbr_med7_r800_description/meshes/collision/link_1.stl" />
                 </geometry>
             </collision>
@@ -95,5 +95,5 @@
                 <origin rpy="0 0 0" xyz="0.0 0.0105 -0.34" />
                 <geometry>
-                    <mesh filename="package://med7_r800_description/meshes/visual/link_2.dae" />
+                    <mesh filename="package://lbr_med7_r800_description/meshes/visual/link_2.dae" />
                 </geometry>
             </visual>
@@ -101,5 +101,5 @@
                 <origin rpy="0 0 0" xyz="0.0 0.0105 -0.34" />
                 <geometry>
-                    <mesh filename="package://med7_r800_description/meshes/collision/link_2.stl" />
+                    <mesh filename="package://lbr_med7_r800_description/meshes/collision/link_2.stl" />
                 </geometry>
             </collision>
@@ -132,5 +132,5 @@
                 <origin rpy="0 0 0" xyz="0.0 0.0 -0.5475" />
                 <geometry>
-                    <mesh filename="package://med7_r800_description/meshes/visual/link_3.dae" />
+                    <mesh filename="package://lbr_med7_r800_description/meshes/visual/link_3.dae" />
                 </geometry>
             </visual>
@@ -138,5 +138,5 @@
                 <origin rpy="0 0 0" xyz="0.0 0.0 -0.5475" />
                 <geometry>
-                    <mesh filename="package://med7_r800_description/meshes/collision/link_3.stl" />
+                    <mesh filename="package://lbr_med7_r800_description/meshes/collision/link_3.stl" />
                 </geometry>
             </collision>
@@ -169,5 +169,5 @@
                 <origin rpy="0 0 0" xyz="0.0 -0.0105 -0.74" />
                 <geometry>
-                    <mesh filename="package://med7_r800_description/meshes/visual/link_4.dae" />
+                    <mesh filename="package://lbr_med7_r800_description/meshes/visual/link_4.dae" />
                 </geometry>
             </visual>
@@ -175,5 +175,5 @@
                 <origin rpy="0 0 0" xyz="0.0 -0.0105 -0.74" />
                 <geometry>
-                    <mesh filename="package://med7_r800_description/meshes/collision/link_4.stl" />
+                    <mesh filename="package://lbr_med7_r800_description/meshes/collision/link_4.stl" />
                 </geometry>
             </collision>
@@ -206,5 +206,5 @@
                 <origin rpy="0 0 0" xyz="0.0 0.0 -0.9475" />
                 <geometry>
-                    <mesh filename="package://med7_r800_description/meshes/visual/link_5.dae" />
+                    <mesh filename="package://lbr_med7_r800_description/meshes/visual/link_5.dae" />
                 </geometry>
             </visual>
@@ -212,5 +212,5 @@
                 <origin rpy="0 0 0" xyz="0.0 0.0 -0.9475" />
                 <geometry>
-                    <mesh filename="package://med7_r800_description/meshes/collision/link_5.stl" />
+                    <mesh filename="package://lbr_med7_r800_description/meshes/collision/link_5.stl" />
                 </geometry>
             </collision>
@@ -243,5 +243,5 @@
                 <origin rpy="0 0 0" xyz="0.0 0.0707 -1.14" />
                 <geometry>
-                    <mesh filename="package://med7_r800_description/meshes/visual/link_6.dae" />
+                    <mesh filename="package://lbr_med7_r800_description/meshes/visual/link_6.dae" />
                 </geometry>
             </visual>
@@ -249,5 +249,5 @@
                 <origin rpy="0 0 0" xyz="0.0 0.0707 -1.14" />
                 <geometry>
-                    <mesh filename="package://med7_r800_description/meshes/collision/link_6.stl" />
+                    <mesh filename="package://lbr_med7_r800_description/meshes/collision/link_6.stl" />
                 </geometry>
             </collision>
@@ -279,5 +279,5 @@
                 <origin rpy="0 0 0" xyz="0.0 0.0 -1.231" />
                 <geometry>
-                    <mesh filename="package://med7_r800_description/meshes/visual/link_7.dae" />
+                    <mesh filename="package://lbr_med7_r800_description/meshes/visual/link_7.dae" />
                 </geometry>
             </visual>
@@ -285,5 +285,5 @@
                 <origin rpy="0 0 0" xyz="0.0 0.0 -1.231" />
                 <geometry>
-                    <mesh filename="package://med7_r800_description/meshes/collision/link_7.stl" />
+                    <mesh filename="package://lbr_med7_r800_description/meshes/collision/link_7.stl" />
                 </geometry>
             </collision>

Commit message: lbr_ prefix

File: urdf/lbr_med7_r800.urdf.xacro (robot description, xacro)
@@ -1,5 +1,5 @@
 <?xml version="1.0"?>
 <!-- top level -->
-<robot name="med7" xmlns:xacro="http://www.ros.org/wiki/xacro">
+<robot name="lbr_med7_r800" xmlns:xacro="http://www.ros.org/wiki/xacro">
     <!-- include the Med 7 R800 macro -->
     <xacro:include filename="$(find lbr_med7_r800_description)/urdf/lbr_med7_r800_macro.xacro" />
@@ -10,5 +10,5 @@
         default="$(find lbr_med7_r800_description)/config/joint_limits.yaml" />
     <!-- Med 7 R800 description -->
-    <xacro:med7_r800
+    <xacro:lbr_med7_r800
         robot_name="$(arg robot_name)"
         joint_limits_path="$(arg joint_limits_path)" />

File: urdf/lbr_med7_r800_macro.xacro (robot description, xacro)
@@ -2,5 +2,5 @@
 <root xmlns:xacro="http://www.ros.org/wiki/xacro">
     <!-- robot as extracted via https://github.com/syuntoku14/fusion2urdf -->
-    <xacro:macro name="med7_r800"
+    <xacro:macro name="lbr_med7_r800"
         params="robot_name:=^|lbr joint_limits_path:=^|'$(find lbr_med7_r800_description)/config/joint_limits.yaml'">
         <!-- load joint limits via yaml -->
